File: KiCAD_project/MP28167_8862_test_board/MP28167_8862_test_board.kicad_pcb (KiCad board)
At the start: 2 copper layers, 3 parts, among them IC1 MP8862GQ-0000-Z, U1 AP63203WU, U2 MP28167GQ-A-Z

Commit message: pcb layout update
Parts:
- added C1: 100u, Capacitor_SMD:CP_Elec_5x5.3, F.Cu at (61.5, 124.9)
- added C10: 22u, Capacitor_SMD:C_0805_2012Metric_Pad1.18x1.45mm_HandSolder, F.Cu at (88.4, 124.9)
- added C11: 22u, Capacitor_SMD:C_0805_2012Metric_Pad1.18x1.45mm_HandSolder, F.Cu at (86.2, 120.8)
- added C12: 22u, Capacitor_SMD:C_0805_2012Metric_Pad1.18x1.45mm_HandSolder, F.Cu at (86.2, 124.9)
- added C13: 22u, Capacitor_SMD:C_0805_2012Metric_Pad1.18x1.45mm_HandSolder, F.Cu at (88.4, 120.8)
- added C14: 22u, Capacitor_SMD:C_0805_2012Metric_Pad1.18x1.45mm_HandSolder, F.Cu at (83.9, 124.9)
- added C15: 100u, Capacitor_SMD:CP_Elec_5x5.3, F.Cu at (93.5, 124.6)
- added C16: 10u, Capacitor_SMD:C_0805_2012Metric_Pad1.18x1.45mm_HandSolder, F.Cu at (112.8, 125.1)
- added C17: 100n, Capacitor_SMD:C_0805_2012Metric_Pad1.18x1.45mm_HandSolder, F.Cu at (115.4, 117.5)
- added C18: 22u, Capacitor_SMD:C_0805_2012Metric_Pad1.18x1.45mm_HandSolder, F.Cu at (117.9, 125.1)
- added C19: 22u, Capacitor_SMD:C_0805_2012Metric_Pad1.18x1.45mm_HandSolder, F.Cu at (117.9, 127.7)
- added C2: 22u, Capacitor_SMD:C_0603_1608Metric_Pad1.08x0.95mm_HandSolder, F.Cu at (67.6, 125.1)
- added C20: 100u, Capacitor_SMD:CP_Elec_5x5.3, F.Cu at (71.8, 95.5)
- added C21: 22u, Capacitor_SMD:C_0805_2012Metric_Pad1.18x1.45mm_HandSolder, F.Cu at (76.4, 95.7)
- added C22: 100n, Capacitor_SMD:C_0603_1608Metric_Pad1.08x0.95mm_HandSolder, F.Cu at (80.5, 95.7)
- added C23: 22n, Capacitor_SMD:C_0603_1608Metric_Pad1.08x0.95mm_HandSolder, F.Cu at (79.6, 98.8)
- added C24: 100n, Capacitor_SMD:C_0805_2012Metric_Pad1.18x1.45mm_HandSolder, F.Cu at (78.9, 91.1)
- added C25: 22n, Capacitor_SMD:C_0603_1608Metric_Pad1.08x0.95mm_HandSolder, F.Cu at (84.3, 100.8)
- added C26: 100n, Capacitor_SMD:C_0805_2012Metric_Pad1.18x1.45mm_HandSolder, F.Cu at (91.6, 91.1)
- added C27: 1u, Capacitor_SMD:C_0603_1608Metric_Pad1.08x0.95mm_HandSolder, F.Cu at (89.8, 98.5)
- added C28: 100n, Capacitor_SMD:C_0603_1608Metric_Pad1.08x0.95mm_HandSolder, F.Cu at (91.6, 95.7)
- added C29: 22u, Capacitor_SMD:C_0805_2012Metric_Pad1.18x1.45mm_HandSolder, F.Cu at (93.8, 95.7)
- added C3: 100n, Capacitor_SMD:C_0805_2012Metric_Pad1.18x1.45mm_HandSolder, F.Cu at (65.6, 125.1)
- added C30: 22u, Capacitor_SMD:C_0805_2012Metric_Pad1.18x1.45mm_HandSolder, F.Cu at (96.5, 95.7)
- added C31: 22u, Capacitor_SMD:C_0805_2012Metric_Pad1.18x1.45mm_HandSolder, F.Cu at (96.5, 91.4)
- added C32: 22u, Capacitor_SMD:C_0805_2012Metric_Pad1.18x1.45mm_HandSolder, F.Cu at (99.0, 95.7)
- added C33: 22u, Capacitor_SMD:C_0805_2012Metric_Pad1.18x1.45mm_HandSolder, F.Cu at (99.0, 91.4)
- added C34: 100u, Capacitor_SMD:CP_Elec_5x5.3, F.Cu at (103.6, 93.7)
- added C4: 22n, Capacitor_SMD:C_0603_1608Metric_Pad1.08x0.95mm_HandSolder, F.Cu at (67.4, 129.7)
- added C5: 100n, Capacitor_SMD:C_0805_2012Metric_Pad1.18x1.45mm_HandSolder, F.Cu at (68.9, 119.3)
- added C6: 22n, Capacitor_SMD:C_0603_1608Metric_Pad1.08x0.95mm_HandSolder, F.Cu at (75.2, 130.2)
- added C7: 100n, Capacitor_SMD:C_0805_2012Metric_Pad1.18x1.45mm_HandSolder, F.Cu at (81.1, 119.3)
- added C8: 1u, Capacitor_SMD:C_0603_1608Metric_Pad1.08x0.95mm_HandSolder, F.Cu at (78.8, 128.2)
- added C9: 100n, Capacitor_SMD:C_0805_2012Metric_Pad1.18x1.45mm_HandSolder, F.Cu at (81.6, 124.9)
- added J1: Conn_01x04_Male, Connector_PinHeader_2.54mm:PinHeader_1x04_P2.54mm_Vertical, F.Cu at (70.4, 135.5)
- added J2: Conn_01x02_Female, Connector_Wire:SolderWire-0.1sqmm_1x02_P3.6mm_D0.4mm_OD1mm, F.Cu at (56.2, 126.9)
- added J3: Conn_01x02_Female, Connector_Wire:SolderWire-0.1sqmm_1x02_P3.6mm_D0.4mm_OD1mm, F.Cu at (98.3, 122.6)
- added J4: Conn_01x02_Female, Connector_Wire:SolderWire-0.1sqmm_1x02_P3.6mm_D0.4mm_OD1mm, F.Cu at (113.4, 131.5)
- added J5: Conn_01x02_Female, Connector_Wire:SolderWire-0.1sqmm_1x02_P3.6mm_D0.4mm_OD1mm, F.Cu at (124.8, 131.5)
- added J6: Conn_01x02_Female, Connector_Wire:SolderWire-0.1sqmm_1x02_P3.6mm_D0.4mm_OD1mm, F.Cu at (67.0, 97.2)
- added J7: Conn_01x02_Female, Connector_Wire:SolderWire-0.1sqmm_1x02_P3.6mm_D0.4mm_OD1mm, F.Cu at (109.2, 91.6)
- added J8: Conn_01x04_Male, Connector_PinHeader_2.54mm:PinHeader_1x04_P2.54mm_Vertical, F.Cu at (76.7, 105.1)
- added L1: 4.7u, footprints:EXL1V0705 inductor, F.Cu at (71.2, 115.0)
- added L2: 4.7u, footprints:SDES064T-4R7MS inductor, F.Cu at (119.2, 120.1)
- added L3: 4.7u, footprints:EXL1V0705 inductor, F.Cu at (81.5, 85.5)
- added R1: 499k, Resistor_SMD:R_0603_1608Metric_Pad0.98x0.95mm_HandSolder, F.Cu at (67.4, 128.2)
- added R10: 0, Resistor_SMD:R_0603_1608Metric_Pad0.98x0.95mm_HandSolder, F.Cu at (88.6, 92.7)
- added R11: 787k, Resistor_SMD:R_0603_1608Metric_Pad0.98x0.95mm_HandSolder, F.Cu at (89.1, 101.0)
- added R12: 430k, Resistor_SMD:R_0603_1608Metric_Pad0.98x0.95mm_HandSolder, F.Cu at (93.1, 100.8)
- added R13: 53.6k, Resistor_SMD:R_0603_1608Metric_Pad0.98x0.95mm_HandSolder, F.Cu at (93.1, 102.6)
- added R2: 499k, Resistor_SMD:R_0603_1608Metric_Pad0.98x0.95mm_HandSolder, F.Cu at (70.2, 130.7)
- added R3: 301k, Resistor_SMD:R_0603_1608Metric_Pad0.98x0.95mm_HandSolder, F.Cu at (71.9, 130.7)
- added R4: 0, Resistor_SMD:R_0603_1608Metric_Pad0.98x0.95mm_HandSolder, F.Cu at (71.7, 121.8)
- added R5: 21.5k, Resistor_SMD:R_0603_1608Metric_Pad0.98x0.95mm_HandSolder, F.Cu at (76.8, 130.2)
- added R6: 0, Resistor_SMD:R_0603_1608Metric_Pad0.98x0.95mm_HandSolder, F.Cu at (78.4, 121.8)
- added R7: 499k, Resistor_SMD:R_0603_1608Metric_Pad0.98x0.95mm_HandSolder, F.Cu at (78.7, 95.7)
- added R8: 0, Resistor_SMD:R_0603_1608Metric_Pad0.98x0.95mm_HandSolder, F.Cu at (82.0, 92.7)
- added R9: 21.5k, Resistor_SMD:R_0603_1608Metric_Pad0.98x0.95mm_HandSolder, F.Cu at (85.9, 100.8)
- added REF**: MountingHole_3.2mm_M3, MountingHole:MountingHole_3.2mm_M3, F.Cu at (129.5, 143.5)
- added REF**: MountingHole_3.2mm_M3, MountingHole:MountingHole_3.2mm_M3, F.Cu at (129.5, 80.0)
- added REF**: MountingHole_3.2mm_M3, MountingHole:MountingHole_3.2mm_M3, F.Cu at (52.6, 143.5)
- added REF**: MountingHole_3.2mm_M3, MountingHole:MountingHole_3.2mm_M3, F.Cu at (52.6, 80.0)
- moved IC1 71.9 mm to (75.0, 125.0)
- moved U2 41.8 mm to (85.3, 95.6)
- moved U1 26.9 mm to (115.4, 121.3)
Routing:
- net Net-(C28-Pad1): track 0.00 -> 40.1 mm, vias 0 -> 2
- net Net-(C18-Pad1): track 0.00 -> 31.2 mm, vias 0 -> 2
- net Net-(C10-Pad1): track 0.00 -> 29.5 mm
- net Net-(C1-Pad1): track 0.00 -> 24.9 mm
- net Net-(C20-Pad1): track 0.00 -> 17.7 mm
- net Net-(C24-Pad1): track 0.00 -> 15.9 mm
- net Net-(C26-Pad1): track 0.00 -> 15.9 mm
- net /Vcc_8862: track 0.00 -> 15.8 mm, vias 0 -> 2
- net Net-(C7-Pad1): track 0.00 -> 14.7 mm
- net Net-(C5-Pad1): track 0.00 -> 14.7 mm
- net /ALT_8862: track 0.00 -> 12.1 mm, vias 0 -> 1
- net Net-(C16-Pad1): track 0.00 -> 12.0 mm
- net /ALT_28167: track 0.00 -> 11.7 mm
- net /SCL_28167: track 0.00 -> 10.6 mm
- net /SDA_8862: track 0.00 -> 10.1 mm
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- added copper zone on B.Cu, net GND
- added copper zone on F.Cu, net GND
- added copper zone on F.Cu, net Net-(C1-Pad1)
- added copper zone on F.Cu, net Net-(C10-Pad1)
- added copper zone on F.Cu, net Net-(C16-Pad1)
- added copper zone on F.Cu, net Net-(C17-Pad2)
- added copper zone on F.Cu, net Net-(C18-Pad1)
- added copper zone on F.Cu, net Net-(C20-Pad1)
- added copper zone on F.Cu, net Net-(C24-Pad1)
- added copper zone on F.Cu, net Net-(C26-Pad1)
- added copper zone on F.Cu, net Net-(C28-Pad1)
- added copper zone on F.Cu, net Net-(C5-Pad1)
- added copper zone on F.Cu, net Net-(C7-Pad1)
- added copper zone on F.Cu, net Net-(IC1-Pad13)
- added copper zone on F.Cu, net Net-(IC1-Pad16)
- added copper zone on F.Cu, net Net-(R10-Pad2)
- added copper zone on F.Cu, net Net-(R8-Pad2)
Other:
- board outline added: 86.8 x 72.2 mm
- board text added: "AP63203"
- board text added: "DC/DC converter test board"
- board text added: "IN"
- board text added: "Krzysztof Sikora"
- board text added: "MP28167"
- board text added: "MP8862"
- board text added: "OUT"
